Commit message: trying some things, dont if working

File: Urdf/leg3dof_ws/src/leg3dof_description/urdf/leg3dof.urdf (robot description, URDF)
Before this commit: robot leg3dof, 1 links, 0 joints
Links:
- removed link base_link
- added link foot_link, mass 0.5; collision cylinder length=0.4 radius=0.025; visual cylinder length=0.4 radius=0.025
- added link hip_link, mass 1.0; collision cylinder length=0.1 radius=0.05; visual cylinder length=0.1 radius=0.05
- added link thigh_link, mass 1.0; collision cylinder length=0.4 radius=0.03; visual cylinder length=0.4 radius=0.03
Joints:
- added joint hip_pitch_joint: type revolute, parent hip_link, child thigh_link, origin xyz=0 0 0 rpy=0 0 0, axis 0 1 0, limit lower=-1.57 upper=1.57 effort=30 velocity=3
- added joint hip_roll_joint: type revolute, parent thigh_link, child foot_link, origin xyz=0 0 -0.4 rpy=0 0 0, axis 1 0 0, limit lower=-1.0 upper=1.0 effort=30 velocity=3
